Commit message: add realsense d435i on it

File: unitree_ros/robots/go2_description/urdf/go2_piper_description.urdf (robot description, URDF)
Before this commit: robot go2_with_piper, 49 links, 48 joints
Links:
- added link realsense_d435, mass 0.15; collision box size=0.1 0.05 0.03; visual mesh filename=package://realsense2_description/meshes/d435.dae scale=1 1 1
Joints:
- added joint realsense_joint: type fixed, parent link6, child realsense_d435, origin xyz=0 0 0.02 rpy=0 0 -1.5708
