Commit message: roamer gazebo setup v1.0

File: unitree_ros/robots/go2_description/xacro/gazebo.xacro (robot description, xacro)
@@ -233,3 +233,52 @@
         <kd  value="1.0"/>
     </gazebo>
+    <gazebo reference="realsense_link">
+        <sensor name="d435i_camera" type="camera">
+            <update_rate>30</update_rate>
+            <camera name="d435i">
+                <horizontal_fov>1.50098</horizontal_fov>
+                <image>
+                    <width>640</width>
+                    <height>480</height>
+                    <format>R8G8B8</format>
+                </image>
+                <clip>
+                    <near>0.1</near>
+                    <far>10.0</far>
+                </clip>
+                <noise>
+                    <type>gaussian</type>
+                    <mean>0.0</mean>
+                    <stddev>0.007</stddev>
+                </noise>
+            </camera>
+            <plugin name="depth_camera" filename="libgazebo_ros_camera.so">
+                <robotNamespace>/</robotNamespace>
+                <depthTopicName>depth/image_raw</depthTopicName>
+                <colorTopicName>color/image_raw</colorTopicName>
+                <ir1TopicName>infra1/image_raw</ir1TopicName>
+                <ir2TopicName>infra2/image_raw</ir2TopicName>
+                <depthInfoTopicName>depth/camera_info</depthInfoTopicName>
+                <colorInfoTopicName>color/camera_info</colorInfoTopicName>
+                <irInfoTopicName>infra/camera_info</irInfoTopicName>
+                <pointCloudTopicName>points</pointCloudTopicName>
+                <updateRate>30.0</updateRate>
+                <depthWidth>640</depthWidth>
+                <depthHeight>480</depthHeight>
+                <colorWidth>640</colorWidth>
+                <colorHeight>480</colorHeight>
+                <baseline>0.05</baseline>
+            </plugin>
+        </sensor>
+    </gazebo>
+    <gazebo reference="d435_Link">
+        <sensor name="d435i_imu" type="imu">
+          <plugin filename="libgazebo_ros_imu_sensor.so" name="d435i_imu_plugin">
+            <topicName>/camera/imu</topicName>
+            <bodyName>d435_Link</bodyName>
+            <updateRate>200.0</updateRate>
+            <frameName>d435_imu_link</frameName>  <!-- 使用唯一框架名 -->
+          </plugin>
+        </sensor>
+    </gazebo>
 </robot>

File: unitree_ros/robots/go2_description/xacro/leg.xacro (robot description, xacro)
@@ -2,6 +2,6 @@
 <robot xmlns:xacro="http://www.ros.org/wiki/xacro">
     <xacro:include filename="$(find go2_description)/xacro/transmission.xacro"/>
-    <xacro:macro name="leg" params="name mirror mirror_dae front_hind front_hind_dae">
-        <joint name="${name}_hip_joint" type="revolute">
+    <xacro:macro name="leg" params="prefix name mirror mirror_dae front_hind front_hind_dae">
+        <joint name="${prefix}${name}_hip_joint" type="revolute">
             <xacro:if value="${(mirror_dae == False) and (front_hind_dae == True)}">
                 <origin rpy="0 0 0" xyz="${leg_offset_x} ${-leg_offset_y} 0"/>
@@ -16,6 +16,6 @@
                 <origin rpy="0 0 0" xyz="${-leg_offset_x} ${leg_offset_y} 0"/>
             </xacro:if>
-            <parent link="trunk"/>
-            <child link="${name}_hip"/>
+            <parent link="${prefix}trunk"/>
+            <child link="${prefix}${name}_hip"/>
             <axis xyz="1 0 0"/>
             <dynamics damping="${damping}" friction="${friction}"/>
@@ -27,5 +27,5 @@
             </xacro:if>
         </joint>
-        <joint name="${name}_hip_rotor_joint" type="fixed">
+        <joint name="${prefix}${name}_hip_rotor_joint" type="fixed">
             <xacro:if value="${(mirror_dae == False) and (front_hind_dae == True)}">
                 <origin rpy="0 0 0" xyz="${hip_rotor_offset_x} ${-hip_rotor_offset_y} 0"/>
@@ -40,8 +40,8 @@
                 <origin rpy="0 0 0" xyz="${-hip_rotor_offset_x} ${hip_rotor_offset_y} 0"/>
             </xacro:if>
-            <parent link="trunk"/>
-            <child link="${name}_hip_rotor"/>
-        </joint>
-        <link name="${name}_hip">
+            <parent link="${prefix}trunk"/>
+            <child link="${prefix}${name}_hip_rotor"/>
+        </joint>
+        <link name="${prefix}${name}_hip">
             <visual>
                 <xacro:if value="${(mirror_dae == True) and (front_hind_dae == True)}">
@@ -77,5 +77,5 @@
             </inertial>
         </link>
-        <link name="${name}_hip_rotor">
+        <link name="${prefix}${name}_hip_rotor">
             <visual>
                 <origin rpy="0 ${PI/2.0} 0" xyz="0 0 0"/>
@@ -100,18 +100,18 @@
             </inertial>
         </link>
-        <joint name="${name}_thigh_joint" type="revolute">
+        <joint name="${prefix}${name}_thigh_joint" type="revolute">
             <origin rpy="0 0 0" xyz="0 ${thigh_offset*mirror} 0"/>
-            <parent link="${name}_hip"/>
-            <child link="${name}_thigh"/>
+            <parent link="${prefix}${name}_hip"/>
+            <child link="${prefix}${name}_thigh"/>
             <axis xyz="0 1 0"/>
             <dynamics damping="${damping}" friction="${friction}"/>
             <limit effort="${thigh_torque_max}" velocity="${thigh_velocity_max}" lower="${thigh_position_min}" upper="${thigh_position_max}"/>
         </joint>
-        <joint name="${name}_thigh_rotor_joint" type="fixed">
+        <joint name="${prefix}${name}_thigh_rotor_joint" type="fixed">
             <origin rpy="0 0 0" xyz="${thigh_rotor_offset_x} ${thigh_rotor_offset_y*mirror} 0"/>
-            <parent link="${name}_hip"/>
-            <child link="${name}_thigh_rotor"/>
-        </joint>
-        <link name="${name}_thigh">
+            <parent link="${prefix}${name}_hip"/>
+            <child link="${prefix}${name}_thigh_rotor"/>
+        </joint>
+        <link name="${prefix}${name}_thigh">
             <visual>
                 <origin rpy="0 0 0" xyz="0 0 0"/>
@@ -141,5 +141,5 @@
             </inertial>
         </link>
-        <link name="${name}_thigh_rotor">
+        <link name="${prefix}${name}_thigh_rotor">
             <visual>
                 <origin rpy="${PI/2.0} 0 0" xyz="0 0 0"/>
@@ -164,18 +164,18 @@
             </inertial>
         </link>
-        <joint name="${name}_calf_joint" type="revolute">
+        <joint name="${prefix}${name}_calf_joint" type="revolute">
             <origin rpy="0 0 0" xyz="0 0 ${-thigh_length}"/>
-            <parent link="${name}_thigh"/>
-            <child link="${name}_calf"/>
+            <parent link="${prefix}${name}_thigh"/>
+            <child link="${prefix}${name}_calf"/>
             <axis xyz="0 1 0"/>
             <dynamics damping="${damping}" friction="${friction}"/>
             <limit effort="${calf_torque_max}" velocity="${calf_velocity_max}" lower="${calf_position_min}" upper="${calf_position_max}"/>
         </joint>
-        <joint name="${name}_calf_rotor_joint" type="fixed">
+        <joint name="${prefix}${name}_calf_rotor_joint" type="fixed">
             <origin rpy="0 0 0" xyz="${calf_rotor_offset_x} ${calf_rotor_offset_y*mirror} 0"/>
-            <parent link="${name}_thigh"/>
-            <child link="${name}_calf_rotor"/>
-        </joint>
-        <link name="${name}_calf">
+            <parent link="${prefix}${name}_thigh"/>
+            <child link="${prefix}${name}_calf_rotor"/>
+        </joint>
+        <link name="${prefix}${name}_calf">
             <visual>
                 <origin rpy="0 0 0" xyz="0 0 0"/>
@@ -200,5 +200,5 @@
             </inertial>
         </link>
-        <link name="${name}_calf_rotor">
+        <link name="${prefix}${name}_calf_rotor">
             <visual>
                 <origin rpy="${PI/2.0} 0 0" xyz="0 0 0"/>
@@ -223,10 +223,10 @@
             </inertial>
         </link>
-        <joint name="${name}_foot_fixed" type="fixed">
+        <joint name="${prefix}${name}_foot_fixed" type="fixed">
             <origin rpy="0 0 0" xyz="0 0 ${-(calf_length)}"/>
-            <parent link="${name}_calf"/>
-            <child link="${name}_foot"/>
-        </joint>
-        <link name="${name}_foot">
+            <parent link="${prefix}${name}_calf"/>
+            <child link="${prefix}${name}_foot"/>
+        </joint>
+        <link name="${prefix}${name}_foot">
             <visual>
                 <origin rpy="0 0 0" xyz="0 0 0"/>
@@ -250,5 +250,5 @@
             </inertial>
         </link>
-        <xacro:leg_transmission name="${name}"/>
+        <xacro:leg_transmission prefix="${prefix}" name="${name}"/>
     </xacro:macro>
 </robot>

File: unitree_ros/robots/go2_description/xacro/materials.xacro (robot description, xacro)
@@ -1,30 +1,36 @@
 <?xml version="1.0"?>
-<robot>
+<robot xmlns:xacro="http://wiki.ros.org/xacro">
+  <!-- 添加包含保护，确保只加载一次 -->
+  <xacro:property name="MATERIALS_XACRO_INCLUDED" value="false"/>
+  <xacro:unless value="${MATERIALS_XACRO_INCLUDED}">
+    <xacro:property name="MATERIALS_XACRO_INCLUDED" value="true"/>
+    <!-- 原始材料定义 -->
     <material name="black">
-        <color rgba="0.0 0.0 0.0 1.0"/>
+      <color rgba="0.0 0.0 0.0 1.0"/>
     </material>
     <material name="blue">
-        <color rgba="0.0 0.0 0.8 1.0"/>
+      <color rgba="0.0 0.0 0.8 1.0"/>
     </material>
     <material name="green">
-        <color rgba="0.0 0.8 0.0 1.0"/>
+      <color rgba="0.0 0.8 0.0 1.0"/>
     </material>
     <material name="grey">
-        <color rgba="0.2 0.2 0.2 0.0"/>
+      <color rgba="0.2 0.2 0.2 0.0"/>
     </material>
     <material name="silver">
-        <color rgba="${233/255} ${233/255} ${216/255} 1.0"/>
+      <color rgba="${233/255} ${233/255} ${216/255} 1.0"/>
     </material>
     <material name="orange">
-        <color rgba="${255/255} ${108/255} ${10/255} 1.0"/>
+      <color rgba="${255/255} ${108/255} ${10/255} 1.0"/>
     </material>
     <material name="brown">
-        <color rgba="${222/255} ${207/255} ${195/255} 1.0"/>
+      <color rgba="${222/255} ${207/255} ${195/255} 1.0"/>
     </material>
     <material name="red">
-        <color rgba="0.8 0.0 0.0 1.0"/>
+      <color rgba="0.8 0.0 0.0 1.0"/>
     </material>
     <material name="white">
-        <color rgba="1.0 1.0 1.0 1.0"/>
+      <color rgba="1.0 1.0 1.0 1.0"/>
     </material>
+  </xacro:unless>
 </robot>

File: unitree_ros/robots/go2_description/xacro/transmission.xacro (robot description, xacro)
@@ -1,31 +1,31 @@
 <?xml version="1.0"?>
 <robot xmlns:xacro="http://www.ros.org/wiki/xacro">
-    <xacro:macro name="leg_transmission" params="name">
-        <transmission name="${name}_hip_tran">
+    <xacro:macro name="leg_transmission" params="prefix name">
+        <transmission name="${prefix}${name}_hip_tran">
             <type>transmission_interface/SimpleTransmission</type>
-            <joint name="${name}_hip_joint">
+            <joint name="${prefix}${name}_hip_joint">
             <hardwareInterface>hardware_interface/EffortJointInterface</hardwareInterface>
             </joint>
-            <actuator name="${name}_hip_motor">
+            <actuator name="${prefix}${name}_hip_motor">
             <hardwareInterface>hardware_interface/EffortJointInterface</hardwareInterface>
             <mechanicalReduction>1</mechanicalReduction>
             </actuator>
         </transmission>
-        <transmission name="${name}_thigh_tran">
+        <transmission name="${prefix}${name}_thigh_tran">
             <type>transmission_interface/SimpleTransmission</type>
-            <joint name="${name}_thigh_joint">
+            <joint name="${prefix}${name}_thigh_joint">
             <hardwareInterface>hardware_interface/EffortJointInterface</hardwareInterface>
             </joint>
-            <actuator name="${name}_thigh_motor">
+            <actuator name="${prefix}${name}_thigh_motor">
             <hardwareInterface>hardware_interface/EffortJointInterface</hardwareInterface>
             <mechanicalReduction>1</mechanicalReduction>
             </actuator>
         </transmission>
-        <transmission name="${name}_calf_tran">
+        <transmission name="${prefix}${name}_calf_tran">
             <type>transmission_interface/SimpleTransmission</type>
-            <joint name="${name}_calf_joint">
+            <joint name="${prefix}${name}_calf_joint">
             <hardwareInterface>hardware_interface/EffortJointInterface</hardwareInterface>
             </joint>
-            <actuator name="${name}_calf_motor">
+            <actuator name="${prefix}${name}_calf_motor">
             <hardwareInterface>hardware_interface/EffortJointInterface</hardwareInterface>
             <mechanicalReduction>1</mechanicalReduction>
